Commit message: Firmware v2.0.0 (I2C link), WT901 IMU and EKF in app 2
Hardware change (2026-10-09): the MCU now talks to the Pi over I2C
(GPIO2/3, level shifter, MCU TWI0 PC4/PC5, address 0x10); the Pi UART on
GPIO14/15 belongs to the new IMU (WT901C-TTL).

Firmware v2.0.0:
- I2C slave. Command 0x01 + vx, vy, w (int16 mm/s, mrad/s) + CRC-8;
  state frame seq, flags, 4 x int32 cumulative counts + CRC-8.
- The TWI ISR does no computation (Pi 4 clock stretching): the main loop
  builds the state frame in a double buffer and checks the command CRC.
- UART only for debug text. Compile check pending (on the Pi).

Pi:
- base_node: smbus2, write and read as two transfers, kernel I2C timeout,
  OSError and CRC errors skipped; speed from the MCU period counter, stamp =
  read time; publish_tf switch; twist covariance for the EKF.
- imu_node + wt901 parser: /imu with the gyro (orientation and acceleration
  covariance -1). scripts/setup_imu.py writes rate and baud into the IMU.
- App 2: robot_localization EKF (wheel vx, vy + IMU turn rate only), the
  EKF publishes TF odom -> base_footprint. imu_link in the URDF.
- setup_pi.sh: PL011 on GPIO14/15 (miniuart-bt, core_freq=250), I2C group,
  robot_localization, smbus2, i2c-tools, gcc-avr.

Tests on the PC: unit tests, firmware frame model test, imu_node with a
fake IMU on a pty, base_node with a fake smbus2 MCU.

Co-Authored-By: Claude Opus 5.5 <noreply@anthropic.com>

File: src/nala_description/urdf/nala.urdf.xacro (robot description, xacro)
@@ -1,5 +1,5 @@
 <?xml version="1.0"?>
 <!--
-  NALA robot frames: base_footprint -> base_link -> laser.
+  NALA robot frames: base_footprint -> base_link -> laser, imu_link.
   All numbers come from config/robot.yaml (xacro argument robot_config).
 -->
@@ -8,4 +8,5 @@
   <xacro:property name="cfg" value="${xacro.load_yaml('$(arg robot_config)')}"/>
   <xacro:property name="laser" value="${cfg['laser']}"/>
+  <xacro:property name="imu" value="${cfg['imu']}"/>
   <!-- On the floor, under the chassis center. Odometry moves this frame. -->
   <link name="base_footprint"/>
@@ -32,3 +33,10 @@
     <origin xyz="${laser['x']} ${laser['y']} ${laser['z']}" rpy="0 0 ${laser['yaw']}"/>
   </joint>
+  <!-- IMU, flat with the chip side up. Published on /tf_static, so the EKF can use /imu. -->
+  <link name="imu_link"/>
+  <joint name="imu_joint" type="fixed">
+    <parent link="base_link"/>
+    <child link="imu_link"/>
+    <origin xyz="${imu['x']} ${imu['y']} ${imu['z']}" rpy="0 0 ${imu['yaw']}"/>
+  </joint>
 </robot>

Commit message: Robot outline with the rod (not centred), wheelbase 335 mm, RPP turn start fix (handover A + B)
A (user answers 2026-10-19: rod as wide as the body, below the LiDAR; sensor on the rod not known yet):
- config/robot.yaml: outline front 0.4425 / back 0.2075 / left, right 0.18 m replaces body_length x
  body_width; read by params.py, coverage_tool/settings.py, the URDF and tools/sim/fake_nala.py.
  Farthest corner 0.478 m: collision radius 0.498 m, plan radius 0.53 m (was 0.293 / 0.33).
- half_wheelbase 0.1675 in config/base.yaml and firmware v2.3.2 (compile-checked on the Pi, not flashed).
- Tests use a fixed test robot (the old centred box): they check the logic, not this robot's size.
B (user chose option A): Nav2 RPP max_angular_accel from its own value controller_angular_accel_rad_s2 3.0
  (first turn step from standstill 0.15 rad/s instead of 0.0175); the velocity gate keeps 0.35 rad/s^2.

Checked: app 3 tests 134/134, base/teleop 55/55, coverage_tool test_sensor 8/8, firmware model tests;
simulation in room Test with a new plan: RETURNED_TO_BASE, 99.9 % covered, 0 contacts.

Co-Authored-By: Claude Opus 5.5 <noreply@anthropic.com>

File: src/nala_description/urdf/nala.urdf.xacro (robot description, xacro)
@@ -9,12 +9,13 @@
   <xacro:property name="laser" value="${cfg['laser']}"/>
   <xacro:property name="imu" value="${cfg['imu']}"/>
+  <xacro:property name="outline" value="${cfg['outline']}"/>
   <!-- On the floor, under the chassis center. Odometry moves this frame. -->
   <link name="base_footprint"/>
-  <!-- Same pose as base_footprint. The flat plate shows the outer size in RViz. -->
+  <!-- Same pose as base_footprint. The flat plate shows the outer outline in RViz (not centred: rod in front). -->
   <link name="base_link">
     <visual>
-      <origin xyz="0 0 0.005"/>
+      <origin xyz="${(outline['front'] - outline['back']) / 2} ${(outline['left'] - outline['right']) / 2} 0.005"/>
       <geometry>
-        <box size="${cfg['body_length']} ${cfg['body_width']} 0.01"/>
+        <box size="${outline['front'] + outline['back']} ${outline['left'] + outline['right']} 0.01"/>
       </geometry>
       <material name="grey">
